File: Hardware/OpenBook.brd (EAGLE design)
At the start: 170.2 x 111.2 mm, 103 parts, among them IC1 BD5229G-TR, IC4 XC6220A331MR-G, J1 FH34SRJ-24S-0.5SH_99_, J2 SAMACSYS_PARTS_USB4110-GF-A, J3 QWIIC_RIGHT_ANGLE, J4 112A-TAAR-R03_ATTEND, Q1 20V/4.2A/52mΩ/1.4W, Q2 20V/4.2A/52mΩ/1.4W, Q3 SI1308EDL-T1-GE3, U1 W25Q512JVEIQ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

Commit message: Polygon pour updated
Routing:
- net GND: track 681.3 -> 725.3 mm, vias 13 -> 42
- net VRTC: track 19.6 -> 25.5 mm
- net RTC_RST: track 64.6 -> 68.2 mm
- net SDA: track 205.6 -> 208.9 mm
- net I2C_PW: track 177.8 -> 181.1 mm
- net MOSI: track 179.8 -> 182.6 mm
- net MISO: track 127.4 -> 130.0 mm
- net 3V3: track 440.5 -> 441.9 mm
